File: kicad/sharprog.sch (KiCad schematic (older format))
At the start: 31 parts, among them J1 Conn_01x11_Male, J2 USB_B_Micro, J3 AudioJack2_SwitchT, J4 AudioJack2_SwitchT, J5 AVR-ISP-6, U1 ATmega328P-AU, U2 FT232RL, Y1 20MHz

Commit message: update kicad
Parts:
- J2: symbol Connector:USB_B_Micro -> sharprog-rescue:USB_B_Micro-Connector
Other:
- moved on the sheet: C1, C2, D1, D2, D3, J1, J3, J4, R1, R2, R3, R7
